File: SCHEMA/JJK-ALIM_COMMUT/commut.kicad_sch (KiCad schematic)
At the start: 0 parts

Commit message: Commutation RX-TX
Parts:
- added C5, C6: 1n, symbol Device:C
- added Q1, Q2, Q4: BSS123, Package_TO_SOT_SMD:SOT-23, symbol Transistor_FET:BSS123
- added Q3: BC857, Package_TO_SOT_SMD:SOT-23, symbol Transistor_BJT:BC857
- added R10: 10, symbol Device:R
- added R11, R13, R14, R4, R5, R6: R, symbol Device:R
- added R12, R2, R3: 10k, symbol Device:R
- added R7, R8: 1M, symbol Device:R
- added R9: 4k7, symbol Device:R
- added U3, U4: BTS50055-1TMA, Package_TO_SOT_SMD:TO-263-7_TabPin4, symbol Power_Management:BTS50055-1TMA
Connections:
- new net: Q3.1 (B), R14.2
- new net: Q4.1 (G), R11.1, R12.1
- new net: C6.1, Q1.1 (G), Q2.3 (D), R10.1, R2.2, R7.1
- new net: C5.1, Q1.3 (D), R3.2, R6.1
- new net: R10.2, U3.3 (IN)
- new net: R4.1, U3.5 (IS)
- new net: R6.2, U4.3 (IN)
- new net: R5.1, U4.5 (IS)
- new net +12V: Q3.2 (E), R13.1
- new net +5V: R2.1, R3.1, R9.1
- new net ANTENNE+12: Q3.3 (C)
- new net COMMUT12V: U3.4 (Vbb), U4.4 (Vbb)
- new net GND: C5.2, C6.2, Q1.2 (S), Q2.2 (S), Q4.2 (S), R11.2, R4.2, R5.2, R7.2, R8.2
- new net PTT: Q2.1 (G), R8.1, R9.2
- new net RX+12V: Q4.3 (D), R13.2, R14.1, U3.1 (OUT), U3.2 (OUT), U3.6 (OUT), U3.7 (OUT)
- new net TX+12V: R12.2, U4.1 (OUT), U4.2 (OUT), U4.6 (OUT), U4.7 (OUT)
Other:
- note added: "10ms"
- note added: "ANT"
- note added: "PTT"
- note added: "RX"
- note added: "TX"
